Commit message: palm updated -> now vertical

File: robot_arm.urdf (robot description, URDF)
Before this commit: robot mediapipe_hand, 11 links, 10 joints
Links:
- link palm: geometry collision box size=0.08 0.1 0.02; visual box size=0.072 0.1 0.02

Commit message: upd: fix limits, WIP on angles alignment

File: robot_arm.urdf (robot description, URDF)
Before this commit: robot mediapipe_hand, 11 links, 10 joints
Links:
- added link base
Joints:
- added joint base_to_palm: type fixed, parent base, child palm, origin xyz=0 0 0.08 rpy=0 0 0
